File: Audio Spektrum Analyser.brd (EAGLE design)
At the start: 160 x 100 mm, 132 parts, among them IC1 LM324N, IC10 LM3914N, IC11 LM3914N, IC12 LM3914N, IC13 LM3914N, IC2 LM324N, IC3 LM324N, IC4 LM3914N, IC5 LM3914N, IC6 LM3914N, IC7 LM3914N, IC8 LM3914N, IC9 LM3914N, M1 ELECTRET_MICROPHON-F6050AP

Commit message: started layout
Parts:
- moved R59 263.9 mm to (150.5, 55.9), turned to 270 degrees
- moved R60 241.4 mm to (150.5, 45.7), turned to 90 degrees
- moved R52 212.4 mm to (94.6, 45.7), turned to 90 degrees
- moved R51 199.9 mm to (94.6, 55.9), turned to 270 degrees
- moved R53 193.8 mm to (108.6, 55.9), turned to 270 degrees
- moved R46 180.2 mm to (52.7, 45.7), turned to 90 degrees
- moved R56 173.2 mm to (122.6, 45.7), turned to 90 degrees
- moved R45 167.6 mm to (52.7, 55.9), turned to 270 degrees
- moved R50 160.7 mm to (80.6, 45.7), turned to 90 degrees
- moved R55 160.1 mm to (122.6, 55.9), turned to 270 degrees
- moved R41 152.4 mm to (24.8, 55.9), turned to 270 degrees
- moved R49 147.6 mm to (80.6, 55.9), turned to 270 degrees
- moved R48 129.5 mm to (66.7, 45.7), turned to 90 degrees
- moved R47 115.9 mm to (66.7, 55.9), turned to 270 degrees
- moved R44 89.5 mm to (38.7, 45.7), turned to 90 degrees
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Routing:
- net +5V: track 0.00 -> 241.4 mm
- net N$87: track 0.00 -> 36.5 mm
- net N$84: track 0.00 -> 36.5 mm
- net N$7: track 0.00 -> 36.5 mm
- net N$61: track 0.00 -> 36.5 mm
- net N$58: track 0.00 -> 36.5 mm
- net N$48: track 0.00 -> 36.5 mm
- net N$99: track 0.00 -> 36.5 mm
- net N$85: track 0.00 -> 36.5 mm
- net N$8: track 0.00 -> 36.5 mm
- net N$60: track 0.00 -> 36.5 mm
- net N$59: track 0.00 -> 36.5 mm
- net N$45: track 0.00 -> 36.5 mm
- net N$100: track 0.00 -> 36.5 mm
- net N$98: track 0.00 -> 36.5 mm
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Other:
- board size 160 x 100 mm -> 228.6 x 136.8 mm

Commit message: connected bandpass
Parts:
- removed R63: 10k, resistor:RTRIM3339P
- added C33, C34, C35: 1u, resistor:E2,5-5
- added C36, C37, C38, C39, C40, C41, C42, C43, C44, C45: 100n, resistor:C050-024X044
- added R4: 47k, rcl:0207/7
- C10: value 1n2 -> 1u; device resistor:C025-024X044 -> resistor:E2,5-5
- C11: value 620p -> 1u; device resistor:C025-024X044 -> resistor:E2,5-5
- C16: value 1u -> 4n7; device resistor:E2,5-5 -> resistor:C025-024X044
- C17: value 1u -> 2n2; device resistor:E2,5-5 -> resistor:C025-024X044
- C18: value 1u -> 1n2; device resistor:E2,5-5 -> resistor:C025-024X044
- C19: value 1u -> 620p; device resistor:E2,5-5 -> resistor:C025-024X044
- C2, C4: value 22n -> 100n; device resistor:C025-024X044 -> resistor:C050-024X044
- C20: value 330p -> 1u; device resistor:C025-024X044 -> resistor:E2,5-5
- C21: value 160p -> 1u; device resistor:C025-024X044 -> resistor:E2,5-5
- C22: value 82p -> 1u; device resistor:C025-024X044 -> resistor:E2,5-5
- C23: value 39p -> 1u; device resistor:C025-024X044 -> resistor:E2,5-5
- C28: value 1u -> 330p; device resistor:E2,5-5 -> resistor:C025-024X044
- C29: value 1u -> 160p; device resistor:E2,5-5 -> resistor:C025-024X044
- C3: value 10n -> 100u; device resistor:C025-024X044 -> resistor:E5-10,5
- C30: value 1u -> 82p; device resistor:E2,5-5 -> resistor:C025-024X044
- C31: value 1u -> 39p; device resistor:E2,5-5 -> resistor:C025-024X044
- C32: value 100u -> 1u; device resistor:E5-10,5 -> resistor:E2,5-5
- C5: value 10n -> 100n; device resistor:C025-024X044 -> resistor:C050-024X044
- C6: value 1u -> 22n; device resistor:E2,5-5 -> resistor:C025-024X044
- C7: value 1u -> 10n; device resistor:E2,5-5 -> resistor:C025-024X044
- C8: value 4n7 -> 22n
- C9: value 2n2 -> 10n
- J1: device Jakobs_LBR:2.5MM-AUX_TH -> Jakobs_LBR:2.5MM-AUX_PC
- R1: value 10k -> 4k7; device rcl:0207/7 -> resistor:RTRIM3339P
- R10, R11: value 1k2 -> 10k; device resistor:0207/7 -> resistor:RTRIM3339P
- R12, R13, R19, R20, R21, R22, R23, R24, R31, R32, R33, R34, R35, R36: value 1k2 -> 120k
- R14, R15, R25, R26, R37, R38: value 1M -> 120k
- R17, R18, R29, R30, R41: value 1k2 -> 1M
- R3: value 4k7 -> 10k; device resistor:RTRIM3339P -> rcl:0207/7
- R42: value 7k5 -> 1M
- R5: value 10k -> 47k
- R61: value 10k -> 1k2; device resistor:RTRIM3339P -> resistor:0207/7
- R62: value 10k -> 7k5; device rcl:0207/7 -> resistor:0207/7
- moved R62 338.4 mm to (187.3, 81.3), turned to 90 degrees
- moved R61 337.9 mm to (187.3, 91.4), turned to 270 degrees
- moved C32 288.8 mm to (144.8, 72.4)
- moved D10 281.8 mm to (167.6, 68.6), turned to 180 degrees
- moved R39 271.2 mm to (160.0, 40.6), turned to 180 degrees
- moved C29 270.7 mm to (184.2, 35.6), turned to 90 degrees
- moved R28 269.7 mm to (139.7, 40.6)
- moved C30 268.3 mm to (184.2, 61.0), turned to 270 degrees
- moved D9 250.2 mm to (153.7, 68.6), turned to 180 degrees
- moved C14 248.1 mm to (135.9, 61.0), turned to 270 degrees
- moved C31 246.2 mm to (156.2, 61.0), turned to 270 degrees
- moved C15 245.6 mm to (123.2, 61.0), turned to 270 degrees
- moved R38 244.3 mm to (167.6, 58.4), turned to 90 degrees
- moved R32 242.5 mm to (188.0, 38.1), turned to 270 degrees
- moved C13 240.9 mm to (135.9, 35.6), turned to 90 degrees
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Connections:
- net +5V: now also C2.1, C36.1, C37.1, C38.1, C39.1, C4.1, C40.1, C41.1, C42.1, C43.1, C44.1, C45.1, C5.1, R1.3, R16.2, R4.2; no longer R14.2, R3.3, R62.2
- net GND: now also C10.-, C11.-, C2.2, C20.-, C21.-, C22.-, C23.-, C32.-, C33.-, C34.-, C35.-, C36.2, C37.2, C38.2, C39.2, C4.2, C40.2, C41.2, C42.2, C43.2, C44.2, C45.2, C5.2, R14.1, R15.1, R25.1, R26.1, R37.1, R38.1, R62.1; no longer C16.-, C17.-, C18.-, C19.-, C28.-, C29.-, C30.-, C31.-, C6.-, C7.-, J1.4, R12.1, R13.1, R21.1, R22.1, R33.1, R34.1, R42.1
- net N$1: now also J1.4, R2.1; no longer J1.2, J1.5, R1.1
- net N$10: now also R11.3; no longer R63.3
- net N$107: now also R43.2; no longer R41.2
- net N$108: now also R43.1, R44.2; no longer R41.1, R42.2
- net N$12: now also C3.+; no longer C1.+
- net N$120: now also R57.2; no longer R55.2
- net N$121: now also R57.1, R58.2; no longer R55.1, R56.2
- net N$125: now also C16.2, R27.2; no longer C12.2, R25.2
- net N$127: now also R59.2; no longer R57.2
- net N$128: now also R59.1, R60.2; no longer R57.1, R58.2
- net N$13: now also C1.+, R1.1; no longer C32.+, R3.1
- net N$130: now also C12.2, R27.1; no longer C8.2, R25.1
- net N$133: now also C8.2, R17.2; no longer C4.2, R15.2
- net N$134: now also C6.2, R17.1; no longer C2.2, R15.1
- net N$135: now also C19.2, R30.2; no longer C15.2, R28.2
- net N$136: now also C6.1, C8.1, R14.2; no longer C2.1, C4.1, R10.2
- net N$138: now also C9.2, R18.2; no longer C5.2, R16.2
- net N$139: now also C7.2, R18.1; no longer C3.2, R16.1
- net N$140: now also C16.1, R19.2, R23.2; no longer C8.1, R17.2, R21.2
- net N$141: now also C7.1, C9.1, R15.2; no longer C3.1, C5.1, R11.2
- net N$144: now also C17.2, R28.2; no longer C13.2, R26.2
- net N$145: now also C13.2, R28.1; no longer C9.2, R26.1
- net N$146: now also C15.2, R30.1; no longer C11.2, R28.1
- net N$147: now also C17.1, R20.2, R24.2; no longer C9.1, R18.2, R22.2
- net N$149: now also C18.2, R29.2; no longer C14.2, R27.2
- net N$150: now also C14.2, R29.1; no longer C10.2, R27.1
- net N$151: now also C28.2, R39.2; no longer C24.2, R37.2
- net N$152: now also C18.1, R21.2, R25.2; no longer C10.1, R19.2, R23.2
- net N$154: now also C19.1, R22.2, R26.2; no longer C11.1, R20.2, R24.2
- net N$156: now also C24.2, R39.1; no longer C20.2, R37.1
- net N$157: now also C28.1, R31.2, R35.2; no longer C20.1, R29.2, R33.2
- net N$159: now also C29.2, R40.2; no longer C25.2, R38.2
- net N$160: now also C25.2, R40.1; no longer C21.2, R38.1
- net N$161: now also C29.1, R32.2, R36.2; no longer C21.1, R30.2, R34.2
- net N$163: now also C30.2, R41.2; no longer C26.2, R39.2
- net N$164: now also C26.2, R41.1; no longer C22.2, R39.1
- net N$165: now also C30.1, R33.2, R37.2; no longer C22.1, R31.2, R35.2
- net N$167: now also C31.2, R42.2; no longer C27.2, R40.2
- net N$168: now also C27.2, R42.1; no longer C23.2, R40.1
- net N$169: now also C31.1, R34.2, R38.2; no longer C23.1, R32.2, R36.2
- net N$179: now also R61.2; no longer R59.2
- net N$180: now also R61.1, R62.2; no longer R59.1, R60.2
- net N$2: now also J1.2, R3.1; no longer J1.3, J1.6, R2.1
- net N$29: now also R47.2; no longer R45.2
- net N$3: now also R3.2; no longer R1.2
- net N$30: now also R47.1, R48.2; no longer R45.1, R46.2
- net N$31: now also R10.1; no longer R61.1
- net N$4: now also C1.-, R4.1; no longer C32.-, R62.1
- net N$42: now also R45.2; no longer R43.2
- net N$43: now also R45.1, R46.2; no longer R43.1, R44.2
- net N$44: now also R11.1; no longer R63.1
- net N$55: now also R49.2; no longer R47.2
- net N$56: now also R49.1, R50.2; no longer R47.1, R48.2
- net N$6: now also R10.3; no longer R61.3
- net N$68: now also R51.2; no longer R49.2
- net N$69: now also R51.1, R52.2; no longer R49.1, R50.2
- net N$81: now also R55.2; no longer R53.2
- net N$82: now also R55.1, R56.2; no longer R53.1, R54.2
- net N$94: now also R53.2; no longer R51.2
- net N$95: now also R53.1, R54.2; no longer R51.1, R52.2
- net OUT1: now also C10.+; no longer C6.+
- net OUT10: now also C35.+; no longer C31.+
- net OUT2: now also C11.+; no longer C7.+
- net OUT3: now also C20.+; no longer C16.+
- net OUT4: now also C21.+; no longer C17.+
- net OUT5: now also C22.+; no longer C18.+
- net OUT6: now also C23.+; no longer C19.+
- net OUT7: now also C32.+; no longer C28.+
- net OUT8: now also C33.+; no longer C29.+
- net OUT9: now also C34.+; no longer C30.+
- net REF: now also R16.1; no longer R14.1
- net VER: now also C3.-, R12.1, R13.1, R21.1, R22.1, R33.1, R34.1; no longer C1.-, R10.1, R11.1, R17.1, R18.1, R29.1, R30.1
Routing:
- net +5V: track 241.4 -> 459.2 mm
- net N$73: track 0.00 -> 36.5 mm
- net N$71: track 0.00 -> 36.5 mm
- net N$171: track 0.00 -> 36.5 mm
- net N$16: track 0.00 -> 36.5 mm
- net N$15: track 0.00 -> 36.5 mm
- net N$14: track 0.00 -> 36.5 mm
- net N$132: track 0.00 -> 36.5 mm
- net N$131: track 0.00 -> 36.5 mm
- net N$112: track 0.00 -> 36.5 mm
- net N$110: track 0.00 -> 36.5 mm
- net N$74: track 0.00 -> 36.5 mm
- net N$20: track 0.00 -> 36.5 mm
- net N$172: track 0.00 -> 36.5 mm
- net N$113: track 0.00 -> 36.5 mm
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- added copper zone on layer 1, net GND
- added copper zone on layer 16, net GND
Other:
- board size 228.6 x 136.8 mm -> 227.3 x 136.8 mm
